Commit message: Refactor Model Name

File: urdf/ExoMy_Model.urdf (robot description, URDF)
Before this commit: robot A01_ExoMy.SLDASM, 5 links, 4 joints
Links:
- link MRB_link: geometry collision mesh filename=package://ExoMy_Model/meshes/MRB_link.STL; visual mesh filename=package://ExoMy_Model/meshes/MRB_link.STL
- link STR_LR_link: geometry collision mesh filename=package://ExoMy_Model/meshes/STR_LR_link.STL; visual mesh filename=package://ExoMy_Model/meshes/STR_LR_link.STL
- link STR_RR_link: geometry collision mesh filename=package://ExoMy_Model/meshes/STR_RR_link.STL; visual mesh filename=package://ExoMy_Model/meshes/STR_RR_link.STL
- link base_link: geometry collision mesh filename=package://ExoMy_Model/meshes/base_link.STL; visual mesh filename=package://ExoMy_Model/meshes/base_link.STL
- link cam_link: geometry collision mesh filename=package://ExoMy_Model/meshes/cam_link.STL; visual mesh filename=package://ExoMy_Model/meshes/cam_link.STL
