Commit message: URDF working except rear wheel starting alignment

File: exomy_model/urdf/exomy_model.urdf (robot description, URDF)
Before this commit: robot exomy_model, 23 links, 22 joints
Joints:
- joint DRV_RR_joint: axis 0 0 1 -> 0 0 -1
- joint STR_LR_joint: origin xyz=0.10378 -0.015418 -0.080775 rpy=1.5708 -1.5708 0 -> xyz=0.10378 -0.015418 -0.080775 rpy=0 -1.5708 -1.5708
- joint STR_RR_joint: origin xyz=-0.103779999964964 -0.0154182000000004 -0.0807754997113281 rpy=1.5707963267949 -1.5707963267949 0 -> xyz=-0.103779999964964 -0.0154182000000004 -0.0807754997113281 rpy=0 -1.5708 -1.5708

Commit message: Fix axis alignment

File: exomy_model/urdf/exomy_model.urdf (robot description, URDF)
Before this commit: robot exomy_model, 23 links, 22 joints
Joints:
- joint DRV_LR_joint: origin xyz=0.0023862 0 -0.057244 rpy=-1.5708 0 1.5708 -> xyz=0.0023862 0 -0.057244 rpy=-1.5708 0 0
- joint DRV_RR_joint: origin xyz=0.00238620000000062 0 -0.05724350028868 rpy=-1.5707963267949 0 1.57079632679492 -> xyz=0 0.00238620000000078 -0.05724350028868 rpy=1.57079634175582 0 0

Commit message: Update transforms to follow lab convention.

File: exomy_model/urdf/exomy_model.urdf (robot description, URDF)
Before this commit: robot exomy_model, 23 links, 22 joints
Joints:
- joint DRV_LR_joint: origin xyz=0.0023862 0 -0.057244 rpy=-1.5708 0 0 -> xyz=0 -0.0023862 -0.057244 rpy=-1.5708 0 0
- joint DRV_RF_joint: axis 0 0 -1 -> 0 0 1
- joint DRV_RM_joint: axis 0 0 -1 -> 0 0 1
- joint DRV_RR_joint: axis 0 0 -1 -> 0 0 1; origin xyz=0 0.00238620000000078 -0.05724350028868 rpy=1.57079634175582 0 0 -> xyz=0 0.00238620000000078 -0.05724350028868 rpy=-1.57079634175582 0 0
- joint MRB_joint: axis 0 0 -1 -> 0 0 1
- joint STR_LR_joint: axis 0 0 -1 -> 0 0 1
- joint STR_RR_joint: axis 0 0 -1 -> 0 0 1

Commit message: Add correct limits to str and bogie joints

File: exomy_model/urdf/exomy_model.urdf (robot description, URDF)
Before this commit: robot exomy_model, 23 links, 22 joints
Joints:
- joint LFB_joint: limit (none) -> lower=-0.47 upper=0.47 effort=0 velocity=0; type continuous -> revolute
- joint MRB_joint: limit lower=-1 upper=1 effort=0 velocity=0 -> lower=-0.47 upper=0.47 effort=0 velocity=0; type continuous -> revolute
- joint RFB_joint: limit lower=0 upper=0 effort=0 velocity=0 -> lower=-0.47 upper=0.47 effort=0 velocity=0; type continuous -> revolute
- joint STR_LF_joint: limit (none) -> lower=-1.57 upper=1.57 effort=0 velocity=0; type continuous -> revolute
- joint STR_LM_joint: limit (none) -> lower=-1.57 upper=1.57 effort=0 velocity=0; type continuous -> revolute
- joint STR_LR_joint: type continuous -> revolute
- joint STR_RF_joint: limit lower=0 upper=0 effort=0 velocity=0 -> lower=-1.57 upper=1.57 effort=0 velocity=0; type continuous -> revolute
- joint STR_RM_joint: limit (none) -> lower=-1.57 upper=1.57 effort=0 velocity=0; type continuous -> revolute
- joint STR_RR_joint: limit lower=0 upper=0 effort=0 velocity=0 -> lower=-1.57 upper=1.57 effort=0 velocity=0; type continuous -> revolute

Commit message: Remove old robot models tests

File: exomy_model/urdf/exomy_model.urdf (robot description, URDF)
Before this commit: robot exomy_model, 23 links, 22 joints
Joints:
- removed joint pupil_right_link
- added joint pupil_right_joint: type fixed, parent eyewhite_link, child pupil_right_link, origin xyz=-0.00026502 -0.0044922 0.002 rpy=0 0 -0.058928, axis 0 0 0

Commit message: Make pupils continuous joints

File: exomy_model/urdf/exomy_model.urdf (robot description, URDF)
Before this commit: robot exomy_model, 23 links, 22 joints
Joints:
- joint pupil_right_joint: axis 0 0 0 -> 0 0 1; type fixed -> continuous
- joint pupils_left_joint: axis 0 0 0 -> 0 0 1; type fixed -> continuous

Commit message: Make pupils move in desired behaviour.

File: exomy_model/urdf/exomy_model.urdf (robot description, URDF)
Before this commit: robot exomy_model, 23 links, 22 joints
Joints:
- removed joint pupils_left_joint
- added joint pupil_left_joint: type continuous, parent eyewhite_link, child pupil_left_link, origin xyz=0.104 0 0.002 rpy=0 0 0, axis 0 0 1
- joint pupil_right_joint: origin xyz=-0.00026502 -0.0044922 0.002 rpy=0 0 -0.058928 -> xyz=0 0 0.002 rpy=0 0 0

Commit message: Make pupils move in sync.

File: exomy_model/urdf/exomy_model.urdf (robot description, URDF)
Before this commit: robot exomy_model, 23 links, 22 joints
Joints:
- joint pupil_right_joint: mimic (none) -> joint=pupil_left_joint
